Commit message: fixed paths

File: urdf/include/gazebo.xacro (robot description, xacro)
@@ -9,5 +9,5 @@
     <leftJoint>base_to_lwheel</leftJoint>
     <rightJoint>base_to_rwheel</rightJoint>
-    <wheelSeparation>0.45</wheelSeparation>
+    <wheelSeparation>0.34</wheelSeparation>
     <wheelDiameter>0.2</wheelDiameter>
     <torque>0.1</torque>
@@ -26,9 +26,9 @@
   </plugin>
 </gazebo>
-<gazebo reference="front_laser">
+<gazebo reference="laser">
   <sensor type="ray" name="head_hokuyo_sensor">
     <pose>0 0 0 0 0 0</pose>
     <visualize>false</visualize>
-    <update_rate>20</update_rate>
+    <update_rate>10</update_rate>
     <ray>
       <scan>
@@ -53,41 +53,8 @@
     <plugin name="gazebo_ros_head_hokuyo_controller" filename="libgazebo_ros_laser.so">
       <topicName>/scan</topicName>
-      <frameName>front_laser</frameName>
+      <frameName>laser</frameName>
     </plugin>
   </sensor>
 </gazebo>
-<!--
-<gazebo reference="rear_laser">
-  <sensor type="ray" name="head_hokuyo_sensor">
-    <pose>0 0 0 0 0 0</pose>
-    <visualize>false</visualize>
-    <update_rate>20</update_rate>
-    <ray>
-      <scan>
-        <horizontal>
-          <samples>720</samples>
-          <resolution>1</resolution>
-          <min_angle>-3.14</min_angle>
-          <max_angle>3.14</max_angle>
-        </horizontal>
-      </scan>
-      <range>
-        <min>0.10</min>
-        <max>10.0</max>
-        <resolution>0.01</resolution>
-      </range>
-      <noise>
-        <type>gaussian</type>
-        <mean>0.0</mean>
-        <stddev>0.01</stddev>
-      </noise>
-    </ray>
-    <plugin name="gazebo_ros_head_hokuyo_controller2" filename="libgazebo_ros_laser.so">
-      <topicName>/rear_laser_scan</topicName>
-      <frameName>rear_laser</frameName>
-    </plugin>
-  </sensor>
-</gazebo>
--->
 <gazebo reference="chassis_frame">
   <visual name="caster_front_visual">
@@ -95,5 +62,5 @@
       <script>
         <uri>file://media/materials/scripts/gazebo.material</uri>
-        <name>Gazebo/Orange</name>
+        <name>Gazebo/Red</name>
       </script>
     </material>
@@ -101,8 +68,31 @@
 </gazebo>
 <gazebo reference="lwheel">
+  <material>Gazebo/Black</material>
+</gazebo>
+<gazebo reference="rwheel">
+  <material>Gazebo/Black</material>
+</gazebo>
+<gazebo reference="caster_rear_collision">
+  <material>Gazebo/Black</material>
+  <mu1>0.001</mu1>
+  <mu2>0.001</mu2>
+</gazebo>
+<gazebo reference="bucket">
   <material>Gazebo/Blue</material>
 </gazebo>
-<gazebo reference="rwheel">
-  <material>Gazebo/Blue</material>
+<gazebo reference="pvc_horizontal">
+  <material>Gazebo/Yellow</material>
+</gazebo>
+<gazebo reference="pvc_up_left">
+  <material>Gazebo/Yellow</material>
+</gazebo>
+<gazebo reference="pvc_up_right">
+  <material>Gazebo/Yellow</material>
+</gazebo>
+<gazebo reference="pvc_45_left">
+  <material>Gazebo/Yellow</material>
+</gazebo>
+<gazebo reference="pvc_45_right">
+  <material>Gazebo/Yellow</material>
 </gazebo>
 </robot>

File: urdf/raptor.urdf.xacro (robot description, xacro)
@@ -1,7 +1,7 @@
 <?xml version="1.0"?>
 	<robot name="raptor" xmlns:xacro="http://www.ros.org/wiki/xacro">
-	<xacro:include filename="$(find raptor_robot)/urdf/include/material.xacro"/>
-	<xacro:include filename="$(find raptor_robot)/urdf/include/gazebo.xacro"/>
-	<xacro:include filename="$(find raptor_robot)/urdf/include/_d435i.urdf.xacro"/>
+	<xacro:include filename="$(find raptor_description)/urdf/include/material.xacro"/>
+	<xacro:include filename="$(find raptor_description)/urdf/include/gazebo.xacro"/>
+	<xacro:include filename="$(find raptor_description)/urdf/include/_d435i.urdf.xacro"/>
   		<link name="base_link">
 		</link>

Commit message: gazebo tuning

File: urdf/include/gazebo.xacro (robot description, xacro)
@@ -66,4 +66,6 @@
     </material>
   </visual>
+  <mu1>0.001</mu1>
+  <mu2>0.001</mu2>
 </gazebo>
 <gazebo reference="lwheel">
@@ -77,4 +79,7 @@
   <mu1>0.001</mu1>
   <mu2>0.001</mu2>
+</gazebo>
+<gazebo reference="caster_rear_visual">
+  <material>Gazebo/Black</material>
 </gazebo>
 <gazebo reference="bucket">

Commit message: LICENSE

File: urdf/include/gazebo.xacro (robot description, xacro)
@@ -10,5 +10,5 @@
     <rightJoint>base_to_rwheel</rightJoint>
     <wheelSeparation>0.34</wheelSeparation>
-    <wheelDiameter>0.2</wheelDiameter>
+    <wheelDiameter>0.28</wheelDiameter>
     <torque>0.1</torque>
     <commandTopic>cmd_vel</commandTopic>
@@ -19,6 +19,6 @@
     <publishOdomTF>true</publishOdomTF>
     <rosDebugLevel>na</rosDebugLevel>
-    <wheelAcceleration>0</wheelAcceleration>
-    <wheelTorque>5</wheelTorque>
+    <wheelAcceleration>20</wheelAcceleration>
+    <wheelTorque>200</wheelTorque>
     <robotBaseFrame>base_link</robotBaseFrame>
     <publishWheelTF>true</publishWheelTF>
@@ -75,11 +75,10 @@
   <material>Gazebo/Black</material>
 </gazebo>
-<gazebo reference="caster_rear_collision">
+<gazebo reference="caster_wheel">
   <material>Gazebo/Black</material>
   <mu1>0.001</mu1>
   <mu2>0.001</mu2>
-</gazebo>
-<gazebo reference="caster_rear_visual">
-  <material>Gazebo/Black</material>
+  <slip1>1.0</slip1>
+  <slip2>1.0</slip2>
 </gazebo>
 <gazebo reference="bucket">

File: urdf/raptor.urdf.xacro (robot description, xacro)
@@ -30,5 +30,17 @@
 			</material>
 			</visual>
+		</link>
+		<joint name="base_to_chassis_frame" type="fixed">
+			<parent link="base_link"/>
+			<child link="chassis_frame"/>
+			<origin xyz="0 0 0.10" rpy="0 0 0"/>
+		</joint>
 			<!-- caster -->
+		<link name="caster_wheel">
+			<inertial>
+    	  		<origin xyz="0 0 0" rpy="0 0 0"/>
+    	  		<mass value="1.0" />
+    	  		<inertia ixx="0.0741666666667" ixy="0.0" ixz="0.0" iyy="0.0585416666667" iyz="0.0" izz="0.0260416666667"/>
+			</inertial>
 			<collision name="caster_rear_collision">
     			<origin rpy=" 0 0 0" xyz="-0.38 0 0.01"/>
@@ -47,5 +59,5 @@
     			</surface>
   			</collision>
-  			<visual name="caster_rear_visual">
+  			<visual>
     			<origin rpy=" 0 0 0" xyz="-0.38 0 0.01"/>
     			<geometry>
@@ -57,8 +69,8 @@
   			</visual>
 		</link>
-		<joint name="base_to_chassis_frame" type="fixed">
-			<parent link="base_link"/>
-			<child link="chassis_frame"/>
-			<origin xyz="0 0 0.10" rpy="0 0 0"/>
+		<joint name="caster_to_chassis_frame" type="fixed">
+			<parent link="chassis_frame"/>
+			<child link="caster_wheel"/>
+			<origin rpy=" 0 0 0" xyz="-0.38 0 0.01"/>
 		</joint>
 		<joint name="imu_joint" type="fixed">
@@ -324,5 +336,5 @@
 			<origin xyz="0.163 0 0.3" rpy="0.0 0.0 3.141592"/>
 			-->
-			<origin xyz="0.40 0.0 0.38" rpy="0.0 0.0 0.0"/>
+			<origin xyz="0.36 0.0 0.35" rpy="0.0 0.0 0.0"/>
 			<axis xyz="0 0 0"/>
 		</joint>

Commit message: now with head

File: urdf/include/gazebo.xacro (robot description, xacro)
@@ -85,4 +85,7 @@
   <material>Gazebo/Blue</material>
 </gazebo>
+<gazebo reference="head">
+  <material>Gazebo/Yellow</material>
+</gazebo>
 <gazebo reference="pvc_horizontal">
   <material>Gazebo/Yellow</material>

File: urdf/raptor.urdf.xacro (robot description, xacro)
@@ -44,5 +44,5 @@
 			</inertial>
 			<collision name="caster_rear_collision">
-    			<origin rpy=" 0 0 0" xyz="-0.38 0 0.01"/>
+    			<origin rpy=" 0 0 0" xyz="0 0 0"/>
     			<geometry>
       				<sphere radius="0.11"/>
@@ -60,5 +60,5 @@
   			</collision>
   			<visual>
-    			<origin rpy=" 0 0 0" xyz="-0.38 0 0.01"/>
+    			<origin rpy=" 0 0 0" xyz="0 0 0"/>
     			<geometry>
       				<sphere radius="0.11"/>
@@ -74,4 +74,34 @@
 			<origin rpy=" 0 0 0" xyz="-0.38 0 0.01"/>
 		</joint>
+		<link name="head">
+			<inertial>
+      			<origin xyz="0 0 0" rpy="0 0 0"/>
+      			<mass value="1.0" />
+      			<inertia ixx="0.0741666666667" ixy="0.0" ixz="0.0" iyy="0.0585416666667" iyz="0.0" izz="0.0260416666667"/>
+			</inertial>
+			<visual>
+				<origin xyz="0 0 0" rpy="0 0 0"/>
+				<geometry>
+					<box size="0.2 0.2 0.1"/>
+				</geometry>
+				<material name="yellow">
+					<color rgba="0 0 0 1"/>
+				</material>
+			</visual>
+			<collision>
+				<origin xyz="0 0 0" rpy="0 0 0"/>
+				<geometry>
+					<box size="0.2 0.2 0.1"/>
+				</geometry>
+			</collision>
+		</link>
+		<joint name="head_to_chassis_frame" type="fixed">
+			<parent link="chassis_frame"/>
+			<child link="head"/>
+			<origin rpy=" 0 0 0" xyz="0.4 0 0.35"/>
+		</joint>
+<!--
+		<link name="imu_link">
+		</link>
 		<joint name="imu_joint" type="fixed">
 			<origin xyz="0.35 0.02 0.39" rpy="0 0 0" />
@@ -79,15 +109,5 @@
 			<child link="imu_link" />
 		</joint>
-		<link name="imu_link">
-		<!--
-		<visual>
-		<origin rpy="0 0 1.5708" xyz="0 0 0"/>
-		<geometry>
-			<mesh filename="package://mpu_6050_driver/mesh/FUGMJ38JX8T7E5A.stl" scale="0.01 0.01 0.01"/>
-		</geometry>
-		<material name="white"/>
-		</visual>
-		-->
-		</link>
+-->
 		<link name="pvc_up_left">
 			<inertial>
@@ -336,5 +356,5 @@
 			<origin xyz="0.163 0 0.3" rpy="0.0 0.0 3.141592"/>
 			-->
-			<origin xyz="0.36 0.0 0.35" rpy="0.0 0.0 0.0"/>
+			<origin xyz="0.35 0.0 0.35" rpy="0.0 0.0 0.0"/>
 			<axis xyz="0 0 0"/>
 		</joint>
@@ -367,5 +387,5 @@
 			<origin xyz="0.163 0 0.3" rpy="0.0 0.0 3.141592"/>
 			-->
-			<origin xyz="0 0.0 0.38" rpy="0.0 0.0 0.0"/>
+			<origin xyz="0 0.0 0.35" rpy="0.0 0.0 0.0"/>
 			<axis xyz="0 0 0"/>
 		</joint>
@@ -398,5 +418,5 @@
 			<origin xyz="0.163 0 0.3" rpy="0.0 0.0 3.141592"/>
 			-->
-			<origin xyz="-0.35 0.0 0.38" rpy="0.0 0.0 0.0"/>
+			<origin xyz="-0.35 0.0 0.35" rpy="0.0 0.0 0.0"/>
 			<axis xyz="0 0 0"/>
 		</joint>
